File: PCB/PCB_EE470/PCB_EE470/PCB_EE470.kicad_pcb (KiCad board)
At the start: 2 copper layers, 68.6 x 53.3 mm, 22 parts, among them IC1 LME49860MAX_NOPB, J1 Power, J2 Digital/PWM, J3 Analog, J4 Digital/PWM

Commit message: pcb good normalement
Parts:
- C1, C2, C3, C4, IC1, MK1, R1, R2, R3, R4, R5, R6, R7, R8: moved to B.Cu
- moved MK1 53.4 mm to (159.1, 77.5)
- moved R7 51.7 mm to (109.7, 68.5)
- moved R8 48.9 mm to (158.7, 67.7)
- moved C3 46.5 mm to (157.5, 72.7), turned to 180 degrees
- moved C4 41.4 mm to (154.9, 63.9), turned to 180 degrees
- moved R1 36.2 mm to (152.3, 72.7), turned to 180 degrees
- moved R6 32.8 mm to (118.1, 68.5), turned to 180 degrees
- moved C2 30.3 mm to (149.3, 76.5)
- moved R3 24.7 mm to (146.5, 65.7), turned to 180 degrees
- moved R4 24.7 mm to (146.5, 69.1), turned to 180 degrees
- moved C1 24.4 mm to (146.3, 72.7), turned to 180 degrees
- moved R2 18.0 mm to (144.6, 76.5), turned to 90 degrees
- moved R5 13.5 mm to (140.7, 65.7), turned to 180 degrees
- moved IC1 5.95 mm to (132.5, 66.3), turned to 180 degrees
Connections:
- C4 pad 1: (no net) -> +5V
- C4 pad 2: (no net) -> GND
- IC1 pad 1: (no net) -> /Out_Etage_1
- IC1 pad 2: (no net) -> Net-(IC1-INVERTING_INPUT_A)
- IC1 pad 3: (no net) -> Net-(IC1-NON-INVERTING_INPUT_A)
- IC1 pad 4: (no net) -> GND
- IC1 pad 5: (no net) -> /Out_Etage_1
- IC1 pad 6: (no net) -> Net-(IC1-INVERTING_INPUT_B)
- IC1 pad 7: (no net) -> /A0
- IC1 pad 8: (no net) -> +5V
- R2 pad 1: (no net) -> GND
- R2 pad 2: (no net) -> Net-(IC1-NON-INVERTING_INPUT_A)
- R3 pad 1: (no net) -> GND
- R3 pad 2: (no net) -> /Out_Etage_1
- R5 pad 1: (no net) -> /Out_Etage_1
- R5 pad 2: (no net) -> Net-(IC1-INVERTING_INPUT_A)
- R6 pad 1: (no net) -> /A0
- R6 pad 2: (no net) -> Net-(IC1-INVERTING_INPUT_B)
- R6 pad 3: (no net) -> Net-(IC1-INVERTING_INPUT_B)
Routing:
- net GND: track 0.00 -> 102.6 mm, vias 0 -> 3
- net /A0: track 0.00 -> 94.1 mm, vias 0 -> 1
- net +5V: track 0.00 -> 56.9 mm, vias 0 -> 1
- net /Out_Etage_1: track 0.00 -> 55.5 mm
- net Net-(IC1-INVERTING_INPUT_B): track 0.00 -> 19.6 mm
- net Net-(IC1-NON-INVERTING_INPUT_A): track 0.00 -> 14.2 mm
- net Net-(C1-Pad1): track 5.12 -> 9.17 mm
- net Net-(IC1-INVERTING_INPUT_A): track 0.00 -> 3.94 mm
- net Net-(MK1-+): track 5.03 -> 6.32 mm

Commit message: pcb good normalement
Parts:
- R2, R5: footprint Capacitor_SMD:C_1206_3216Metric_Pad1.33x1.80mm_HandSolder -> Resistor_SMD:R_0805_2012Metric_Pad1.20x1.40mm_HandSolder
- R3, R4, R7, R8: footprint Capacitor_SMD:C_1206_3216Metric_Pad1.33x1.80mm_HandSolder -> Resistor_SMD:R_1206_3216Metric_Pad1.30x1.75mm_HandSolder
- R6: footprint Potentiometer_SMD:Potentiometer_ACP_CA6-VSMD_Vertical_Hole -> Potentiometer_THT:Potentiometer_Vishay_T73XW_Horizontal
- moved R6 3.99 mm to (120.9, 65.7), turned to 90 degrees
- moved R8 0.54 mm to (158.9, 68.2)
- moved MK1 0.45 mm to (159.1, 78.0)
Routing:
- net GND: track 102.6 -> 1.95 mm, vias 3 -> 0
- net +5V: track 56.9 -> 106.0 mm
- net /Out_Etage_1: track 55.5 -> 22.0 mm
- net Net-(IC1-INVERTING_INPUT_B): track 19.6 -> 31.6 mm
- net /A0: track 94.1 -> 88.5 mm
- added copper zone on F.Cu, net GND
Other:
- board size 68.6 x 53.3 mm -> 68.6 x 53.4 mm

Commit message: pcb good normalement
Parts:
- added TP101: Out1, TestPoint:TestPoint_Loop_D3.80mm_Drill2.0mm, F.Cu at (148.9, 58.6)
- added TP102: Out2, TestPoint:TestPoint_Loop_D3.80mm_Drill2.0mm, F.Cu at (140.6, 58.6)
- added Tp103: Out3, TestPoint:TestPoint_Loop_D3.80mm_Drill2.0mm, F.Cu at (119.8, 58.8)
Routing:
- net /Out_Etage_1: track 22.0 -> 39.7 mm
- net Net-(C3-Pad2): track 2.05 -> 18.2 mm
- net /A0: track 88.5 -> 75.5 mm, vias 1 -> 0
