File: PCB/PCB_EE470/PCB_EE470/PCB_EE470.kicad_sch (KiCad schematic)
At the start: 18 parts, among them IC1 LME49860MAX_NOPB, J1 Power, J2 Digital/PWM, J3 Analog, J4 Digital/PWM

Commit message: pcb good normalement
Parts:
- R2, R5: footprint Capacitor_SMD:C_1206_3216Metric_Pad1.33x1.80mm_HandSolder -> Resistor_SMD:R_0805_2012Metric_Pad1.20x1.40mm_HandSolder
- R3, R4, R7, R8: footprint Capacitor_SMD:C_1206_3216Metric_Pad1.33x1.80mm_HandSolder -> Resistor_SMD:R_1206_3216Metric_Pad1.30x1.75mm_HandSolder
- R6: footprint Potentiometer_SMD:Potentiometer_ACP_CA6-VSMD_Vertical_Hole -> Potentiometer_THT:Potentiometer_Vishay_T73XW_Horizontal
Changed lines of the file:
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@@
       (effects (font (size 1.27 1.27)) (justify left))
     )
-    (property "Footprint" "Capacitor_SMD:C_1206_3216Metric_Pad1.33x1.80mm_HandSolder" (at 88.392 120.65 90)
+    (property "Footprint" "Resistor_SMD:R_1206_3216Metric_Pad1.30x1.75mm_HandSolder" (at 88.392 120.65 90)
       (effects (font (size 1.27 1.27)) hide)
     )
@@
       (effects (font (size 1.27 1.27)))
     )
-    (property "Footprint" "Capacitor_SMD:C_1206_3216Metric_Pad1.33x1.80mm_HandSolder" (at 154.178 134.62 90)
+    (property "Footprint" "Resistor_SMD:R_0805_2012Metric_Pad1.20x1.40mm_HandSolder" (at 154.178 134.62 90)
       (effects (font (size 1.27 1.27)) hide)
     )
@@
       (effects (font (size 1.27 1.27)))
     )
-    (property "Footprint" "Capacitor_SMD:C_1206_3216Metric_Pad1.33x1.80mm_HandSolder" (at 156.21 122.428 90)
+    (property "Footprint" "Resistor_SMD:R_1206_3216Metric_Pad1.30x1.75mm_HandSolder" (at 156.21 122.428 90)
       (effects (font (size 1.27 1.27)) hide)
     )
@@
       (effects (font (size 1.27 1.27)))
     )
-    (property "Footprint" "Capacitor_SMD:C_1206_3216Metric_Pad1.33x1.80mm_HandSolder" (at 172.72 118.618 90)
+    (property "Footprint" "Resistor_SMD:R_0805_2012Metric_Pad1.20x1.40mm_HandSolder" (at 172.72 118.618 90)
       (effects (font (size 1.27 1.27)) hide)
     )
@@
       (effects (font (size 1.27 1.27)))
     )
-    (property "Footprint" "Capacitor_SMD:C_1206_3216Metric_Pad1.33x1.80mm_HandSolder" (at 156.21 118.618 90)
+    (property "Footprint" "Resistor_SMD:R_1206_3216Metric_Pad1.30x1.75mm_HandSolder" (at 156.21 118.618 90)
       (effects (font (size 1.27 1.27)) hide)
     )
@@
       (effects (font (size 1.27 1.27)))
     )
-    (property "Footprint" "Capacitor_SMD:C_1206_3216Metric_Pad1.33x1.80mm_HandSolder" (at 270.51 118.618 90)
+    (property "Footprint" "Resistor_SMD:R_1206_3216Metric_Pad1.30x1.75mm_HandSolder" (at 270.51 118.618 90)
       (effects (font (size 1.27 1.27)) hide)
     )
@@
       (effects (font (size 1.27 1.27)))
     )
-    (property "Footprint" "Potentiometer_SMD:Potentiometer_ACP_CA6-VSMD_Vertical_Hole" (at 256.54 116.84 0)
-      (effects (font (size 1.27 1.27)) hide)
-    )
+    (property "Footprint" "Potentiometer_THT:Potentiometer_Vishay_T73XW_Horizontal" (at 256.54 116.84 0)
+      (effects (font (size 1.27 1.27)) hide)
+    )

Commit message: pcb good normalement
Parts:
- added TP101: Out1, TestPoint:TestPoint_Loop_D3.80mm_Drill2.0mm, symbol Connector:TestPoint
- added TP102: Out2, TestPoint:TestPoint_Loop_D3.80mm_Drill2.0mm, symbol Connector:TestPoint
- added Tp103: Out3, TestPoint:TestPoint_Loop_D3.80mm_Drill2.0mm, symbol Connector:TestPoint
Connections:
- net A0: now also Tp103.1
- net Out_Etage_1: now also TP102.1
- net at C3.2, R1.1: now also TP101.1
Changed lines of the file:
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@@
   (junction (at 152.4 127) (diameter 0) (color 0 0 0 0)
   )
+  (junction (at 108.585 127) (diameter 0) (color 0 0 0 0)
+  )
   (junction (at 144.78 127) (diameter 0) (color 0 0 0 0)
   )
@@
   (junction (at 90.17 127) (diameter 0) (color 0 0 0 0)
   )
+  (junction (at 255.27 107.95) (diameter 0) (color 0 0 0 0)
+  )
   (junction (at 262.89 116.84) (diameter 0) (color 0 0 0 0)
+  )
+  (junction (at 252.73 121.92) (diameter 0) (color 0 0 0 0)
   )
   (no_connect (at 238.76 24.13))
@@
     (stroke (width 0) (type default))
   )
+  (wire (pts (xy 252.73 121.92) (xy 256.54 121.92))
+    (stroke (width 0) (type default))
+  )
   (wire (pts (xy 144.78 127) (xy 144.78 120.65))
     (stroke (width 0) (type default))
@@
     (stroke (width 0) (type solid))
   )
-  (wire (pts (xy 104.14 127) (xy 119.38 127))
+  (wire (pts (xy 104.14 127) (xy 108.585 127))
     (stroke (width 0) (type default))
   )
@@
     (stroke (width 0) (type default))
   )
-  (wire (pts (xy 252.73 107.95) (xy 260.35 107.95))
+  (wire (pts (xy 252.73 107.95) (xy 255.27 107.95))
+    (stroke (width 0) (type default))
+  )
+  (wire (pts (xy 274.32 116.84) (xy 276.86 116.84))
     (stroke (width 0) (type default))
   )
@@
     (stroke (width 0) (type default))
   )
+  (wire (pts (xy 255.27 107.95) (xy 260.35 107.95))
+    (stroke (width 0) (type default))
+  )
   (wire (pts (xy 248.92 116.84) (xy 252.73 116.84))
     (stroke (width 0) (type default))
@@
     (stroke (width 0) (type default))
   )
-  (wire (pts (xy 274.32 116.84) (xy 276.86 116.84))
-    (stroke (width 0) (type default))
-  )
   (wire (pts (xy 269.24 26.67) (xy 269.24 44.45))
     (stroke (width 0) (type solid))
@@
     (stroke (width 0) (type default))
   )
-  (wire (pts (xy 248.92 121.92) (xy 256.54 121.92))
+  (wire (pts (xy 248.92 121.92) (xy 252.73 121.92))
     (stroke (width 0) (type default))
   )
@@
     (stroke (width 0) (type default))
   )
+  (wire (pts (xy 108.585 124.46) (xy 108.585 127))
+    (stroke (width 0) (type default))
+  )
   (wire (pts (xy 266.7 57.15) (xy 279.4 57.15))
     (stroke (width 0) (type solid))
@@
   (wire (pts (xy 226.06 59.69) (xy 238.76 59.69))
     (stroke (width 0) (type solid))
+  )
+  (wire (pts (xy 108.585 127) (xy 119.38 127))
+    (stroke (width 0) (type default))
   )
   (wire (pts (xy 152.4 139.7) (xy 152.4 138.43))
@@
     )
   )
+  (symbol (lib_id "Connector:TestPoint") (at 252.73 121.92 180) (unit 1)
+    (in_bom yes) (on_board yes) (dnp no) (fields_autoplaced)
+    (property "Reference" "TP102" (at 255.27 123.952 0)
+      (effects (font (size 1.27 1.27)) (justify right))
+    )
+    (property "Value" "Out2" (at 255.27 126.492 0)
+      (effects (font (size 1.27 1.27)) (justify right))
+    )
+    (property "Footprint" "TestPoint:TestPoint_Loop_D3.80mm_Drill2.0mm" (at 247.65 121.92 0)
+      (effects (font (size 1.27 1.27)) hide)
+    )
+    (property "Datasheet" "~" (at 247.65 121.92 0)
+      (effects (font (size 1.27 1.27)) hide)
+    )
+    (pin "1")
+    (instances
+      (project "PCB_EE470"
+        (path "/e63e39d7-6ac0-4ffd-8aa3-1841a4541b55"
+          (reference "TP102") (unit 1)
+        )
+      )
+    )
+  )
+  (symbol (lib_id "Connector:TestPoint") (at 255.27 107.95 0) (unit 1)
+    (in_bom yes) (on_board yes) (dnp no)
+    (property "Reference" "Tp103" (at 254.635 99.695 0)
+      (effects (font (size 1.27 1.27)) (justify left))
+    )
+    (property "Value" "Out3" (at 254.635 102.235 0)
+      (effects (font (size 1.27 1.27)) (justify left))
+    )
+    (property "Footprint" "TestPoint:TestPoint_Loop_D3.80mm_Drill2.0mm" (at 260.35 107.95 0)
+      (effects (font (size 1.27 1.27)) hide)
+    )
+    (property "Datasheet" "~" (at 260.35 107.95 0)
+      (effects (font (size 1.27 1.27)) hide)
+    )
+    (pin "1")
+    (instances
+      (project "PCB_EE470"
+        (path "/e63e39d7-6ac0-4ffd-8aa3-1841a4541b55"
+          (reference "Tp103") (unit 1)
+        )
+      )
+    )
+  )
   (symbol (lib_id "Device:C") (at 148.59 127 90) (unit 1)
     (in_bom yes) (on_board yes) (dnp no)
@@
         )
       )
+    )
+  )
+  (symbol (lib_id "Connector:TestPoint") (at 108.585 124.46 0) (unit 1)
+    (in_bom yes) (on_board yes) (dnp no)
+    (property "Reference" "TP101" (at 109.22 114.935 0)
+      (effects (font (size 1.27 1.27)) (justify left))
+    )
+    (property "Value" "Out1" (at 108.585 118.11 0)
+      (effects (font (size 1.27 1.27)) (justify left))
+    )
+    (property "Footprint" "TestPoint:TestPoint_Loop_D3.80mm_Drill2.0mm" (at 113.665 124.46 0)
+      (effects (font (size 1.27 1.27)) hide)
+    )
+    (property "Datasheet" "~" (at 113.665 124.46 0)
+      (effects (font (size 1.27 1.27)) hide)
+    )
+    (pin "1")
+    (instances
+      (project "PCB_EE470"
+        (path "/e63e39d7-6ac0-4ffd-8aa3-1841a4541b55"
+          (reference "TP101") (unit 1)
+        )
+      )
